Commit message: fix logging, add lidar to urdf

File: kris_robot/urdf/kris_robot.urdf (robot description, URDF)
Before this commit: robot kris_robot, 3 links, 2 joints
Links:
- added link laser_frame, mass 0.05; visual cylinder length=0.034 radius=0.035
- link base_link: mass None -> 0.25
- link lwheel: mass None -> 0.1
- link rwheel: mass None -> 0.1
Joints:
- added joint laser_joint: type fixed, parent base_link, child laser_frame, origin xyz=0.1 0 0.175 rpy=0 0 0
- joint base_link_to_lwheel: type continuous -> fixed
- joint base_link_to_rwheel: type continuous -> fixed

Commit message: update urdf of the robot

File: kris_robot/urdf/kris_robot.urdf (robot description, URDF)
Before this commit: robot kris_robot, 4 links, 3 joints
Links:
- removed link base_link
- added link kris_robot1_base_link, mass 0.25; visual cylinder length=0.08 radius=0.055
Joints:
- removed joint base_link_to_lwheel
- removed joint base_link_to_rwheel
- added joint kris_robot1_base_link_to_lwheel: type continuous, parent kris_robot1_base_link, child lwheel, origin xyz=0.050 0 0.02 rpy=1.5708 1.5708 0, axis 
- added joint kris_robot1_base_link_to_rwheel: type continuous, parent kris_robot1_base_link, child rwheel, origin xyz=-0.050 0 0.02 rpy=1.5708 1.5708 0, axis 
- joint laser_joint: parent base_link -> kris_robot1_base_link

Commit message: update urdf

File: kris_robot/urdf/kris_robot.urdf (robot description, URDF)
Before this commit: robot kris_robot1, 4 links, 3 joints
Links:
- removed link laser_frame
- added link kris_robot1_laser_frame, mass 0.05; visual cylinder length=0.034 radius=0.035
Joints:
- joint laser_joint: child laser_frame -> kris_robot1_laser_frame

Commit message: update urdf

File: kris_robot/urdf/kris_robot.urdf (robot description, URDF)
Before this commit: robot kris_robot1, 4 links, 3 joints
Links:
- removed link lwheel
- removed link rwheel
- added link kris_robot1_lwheel, mass 0.1; visual cylinder length=0.025 radius=0.0325
- added link kris_robot1_rwheel, mass 0.1; visual cylinder length=0.025 radius=0.0325
Joints:
- removed joint kris_robot1_base_link_to_lwheel
- removed joint kris_robot1_base_link_to_rwheel
- added joint kris_robot1_base_link_to_kris_robot1_lwheel: type continuous, parent kris_robot1_base_link, child kris_robot1_lwheel, origin xyz=0.050 0 0.02 rpy=1.5708 1.5708 0, axis 
- added joint kris_robot1_base_link_to_kris_robot1_rwheel: type continuous, parent kris_robot1_base_link, child kris_robot1_rwheel, origin xyz=-0.050 0 0.02 rpy=1.5708 1.5708 0, axis 
