Commit message: increase spin timeout

File: robot_sim/urdf/robot.urdf (robot description, URDF)
Before this commit: robot robot, 3 links, 2 joints
Links:
- removed link base_link
- added link kris_robot1_base_link; visual cylinder length=0.08 radius=0.055
Joints:
- removed joint base_link_to_lwheel
- removed joint base_link_to_rwheel
- added joint kris_robot1_base_link_to_lwheel: type continuous, parent kris_robot1_base_link, child lwheel, origin xyz=0.050 0 0.02 rpy=1.5708 1.5708 0
- added joint kris_robot1_base_link_to_rwheel: type continuous, parent kris_robot1_base_link, child rwheel, origin xyz=-0.050 0 0.02 rpy=1.5708 1.5708 0
